File: pcb/v0/PERIPH/PERIPH.kicad_pcb (KiCad board)
At the start: 4 copper layers, 35 x 35 mm, 65 parts, among them J1 JST SH 4 pin, J2 JST SH 4 pin, J3 Conn_01x02_Socket, J4 Conn_01x02_Socket, J6 Conn_01x02_Socket, M1 Conn_01x02_Socket, M2 Conn_01x02_Socket, M3 Conn_01x02_Socket, U1 DRV8234RTER, U10 MCP4725A1T-E/CH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

Commit message: finish PERIPH V0
Parts:
- R12: footprint Resistor_SMD:R_0603_1608Metric -> Resistor_SMD:R_2512_6332Metric
- moved C5 5.54 mm to (124.7, 64.4), turned to 0 degrees
- moved R7 1.78 mm to (124.4, 75.5)
- moved C19 0.68 mm to (124.3, 77.0)
- moved R12 0.54 mm to (124.7, 69.9)
- renumbered M3 to J10, 12V to J5, BAT to J7, M1 to J8, M2 to J9
Routing:
- net Net-(U4-IPROPI): track 22.0 -> 27.5 mm
- net Voltage Out: track 66.4 -> 65.2 mm
- net GND: track 120.6 -> 119.4 mm
- net SCL: track 84.7 -> 85.8 mm
Other:
- board text added: "PERIPH REV 0"
- board text removed: "PERIPH REV0"
