File: pcb/v0/PERIPH/PERIPH.kicad_sch (KiCad schematic)
At the start: 64 parts, among them J1 JST SH 4 pin, J10 Conn_01x02_Socket, J2 JST SH 4 pin, J3 Conn_01x02_Socket, J4 Conn_01x02_Socket, J5 Conn_01x02_Socket, J6 Conn_01x02_Socket, J7 Conn_01x02_Socket, J8 Conn_01x02_Socket, J9 Conn_01x02_Socket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

Commit message: finish PERIPH V0
Parts:
- C1, C14, C19, C2, C6, C7: MPN (none) -> CL10B105KP8NNNC; Manufacturer (none) -> Samsung Electro-Mechanics; VPN (none) -> 1276-1946-1-ND; Vendor (none) -> DigiKey
- C10, C11, C15, C16, C20, C21: MPN (none) -> CL32B226KAJNNNE; Manufacturer (none) -> Samsung Electro-Mechanics; VPN (none) -> 1276-3392-1-ND; Vendor (none) -> DigiKey
- C12, C17, C9: MPN (none) -> TMK212AB7475KG-T; Manufacturer (none) -> Taiyo Yuden; VPN (none) -> 587-2990-1-ND; Vendor (none) -> DigiKey
- C13, C18, C23, C24, C27, C28, C31, C4, C5, C8: MPN (none) -> C0603C104K3RACTU; Manufacturer (none) -> KEMET; VPN (none) -> 399-C0603C104K3RACTUCT-ND; Vendor (none) -> DigiKey
- C22, C29, C30: MPN (none) -> KTS250B476M76N0T00; Manufacturer (none) -> Chemi-Con; VPN (none) -> 565-4695-1-ND; Vendor (none) -> DigiKey
- C3: MPN (none) -> EEH-ZA1H101P; Manufacturer (none) -> Panasonic Electronic Components; VPN (none) -> P15442CT-ND; Vendor (none) -> DigiKey
- J1, J2: MPN (none) -> SM04B-SRSS-TB; Manufacturer (none) -> JST Sales America Inc.; VPN (none) -> 455-SM04B-SRSS-TBCT-ND; Vendor (none) -> DigiKey
- J10, J3, J4, J5, J6, J7, J8, J9: Vendor (none) -> DigiKey; now not fitted
- R10, R9: MPN (none) -> CR0603-FX-2201ELF; Manufacturer (none) -> Bourns Inc.; VPN (none) -> 118-CR0603-FX-2201ELFCT-ND; Vendor (none) -> DigiKey
- R12: footprint Resistor_SMD:R_0603_1608Metric -> Resistor_SMD:R_2512_6332Metric; MPN (none) -> HoCG25122R050A4; Manufacturer (none) -> Shenzhen Milliohm Electronic Co.,Ltd; VPN (none) -> 5705-HoCG25122R050A4TR-ND; Vendor (none) -> DigiKey
- R13: MPN (none) -> RC0603FR-0723K2L; Manufacturer (none) -> YAGEO; VPN (none) -> 311-23.2KHRCT-ND; Vendor (none) -> DigiKey
- R14, R16, R18, R20, R23, R5: MPN (none) -> RC0603FR-0710KL; Manufacturer (none) -> YAGEO; VPN (none) -> 311-10.0KHRCT-ND; Vendor (none) -> DigiKey
- R15: MPN (none) -> RC0603FR-0740K2L; Manufacturer (none) -> YAGEO; VPN (none) -> 311-40.2KHRCT-ND; Vendor (none) -> DigiKey
- R17: MPN (none) -> CRCW0603110KFKEAC; Manufacturer (none) -> Vishay Dale; VPN (none) -> 541-5140-1-ND; Vendor (none) -> DigiKey
- R19, R24, R7: MPN (none) -> CR0603-JW-472ELF; Manufacturer (none) -> Bourns Inc.; VPN (none) -> CR0603-JW-472ELFCT-ND; Vendor (none) -> DigiKey
- U1, U2, U4: MPN (none) -> DRV8234RTER; Manufacturer (none) -> Texas Instruments; VPN (none) -> 296-DRV8234RTERCT-ND; Vendor (none) -> DigiKey
- U10, U3: MPN (none) -> MCP4725A1T-E/CH; Manufacturer (none) -> Microchip Technology; VPN (none) -> MCP4725A1T-E/CHCT-ND; Vendor (none) -> DigiKey
- U5, U7, U8: MPN (none) -> TPSM33625RDNR; Manufacturer (none) -> Texas Instruments; VPN (none) -> 296-TPSM33625RDNRCT-ND; Vendor (none) -> DigiKey
- U6: MPN (none) -> MCP4725A2T-E/CH; Manufacturer (none) -> Microchip Technology; VPN (none) -> MCP4725A2T-E/CHCT-ND; Vendor (none) -> DigiKey
- U9: MPN (none) -> INA219BIDCNT; Manufacturer (none) -> Texas Instruments; VPN (none) -> 296-27898-1-ND; Vendor (none) -> DigiKey
